File: level 1/level_1_light_maze/light_maze.kicad_sch (KiCad schematic)
At the start: 35 parts, among them J1 Conn_01x02_Socket, J2 Conn_01x03_Socket, J3 Conn_01x03_Socket, J4 Conn_01x03_Socket, J5 Conn_01x03_Socket, J6 Conn_01x03_Socket, J7 Conn_01x03_Socket, J8 Conn_01x03_Socket, J9 Conn_01x03_Socket, U2 LM339

Commit message: pcb update
Other:
- moved on the sheet: J2, J3, J4, R11, R12, R13, R22
