File: level 1/level_1_light_maze/light_maze.kicad_pcb (KiCad board)
At the start: 2 copper layers, 90 x 33 mm, 35 parts, among them J1 Conn_01x02_Socket, J2 Conn_01x03_Socket, J3 Conn_01x03_Socket, J4 Conn_01x03_Socket, J5 Conn_01x03_Socket, J6 Conn_01x03_Socket, J7 Conn_01x03_Socket, J8 Conn_01x03_Socket, J9 Conn_01x03_Socket, U2 LM339

Commit message: pcb changes
Parts:
- moved R18 19.7 mm to (139.0, 116.0)
- moved R16 19.0 mm to (139.0, 113.0)
- moved R13 19.0 mm to (130.9, 113.0)
- moved R17 18.1 mm to (139.9, 108.0)
- moved R12 15.6 mm to (130.9, 116.0)
- moved R9 10.4 mm to (130.9, 119.0)
- moved J1 9.51 mm to (131.0, 95.0)
- moved R11 7.07 mm to (151.0, 113.0)
- moved R6 6.54 mm to (128.0, 114.1)
- moved R10 5.42 mm to (130.9, 122.0)
- moved U2 4.90 mm to (135.0, 106.0)
- moved R5 4.12 mm to (128.0, 107.1)
- moved R7 2.20 mm to (132.0, 99.0)
- moved R4 1.41 mm to (128.0, 95.0)
- moved R21 0.54 mm to (186.0, 115.0)
Other:
- board size 90 x 33 mm -> 88 x 33 mm
Changed lines of the file:
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@@
 	(footprint "Resistor_THT:R_Axial_DIN0204_L3.6mm_D1.6mm_P5.08mm_Horizontal"
 		(layer "F.Cu")
-		(at 185.46 115)
+		(at 186 115)
 		(descr "Resistor, Axial_DIN0204 series, Axial, Horizontal, pin pitch=5.08mm, 0.167W, length*diameter=3.6*1.6mm^2, http://cdn-reichelt.de/documents/datenblatt/B400/1_4W%23YAG.pdf")
 		(tags "Resistor Axial_DIN0204 series Axial Horizontal pin pitch 5.08mm 0.167W length 3.6mm diameter 1.6mm")
@@
 	(footprint "Resistor_THT:R_Axial_DIN0204_L3.6mm_D1.6mm_P5.08mm_Horizontal"
 		(layer "F.Cu")
-		(at 146 112)
+		(at 130.92 116)
 		(descr "Resistor, Axial_DIN0204 series, Axial, Horizontal, pin pitch=5.08mm, 0.167W, length*diameter=3.6*1.6mm^2, http://cdn-reichelt.de/documents/datenblatt/B400/1_4W%23YAG.pdf")
 		(tags "Resistor Axial_DIN0204 series Axial Horizontal pin pitch 5.08mm 0.167W length 3.6mm diameter 1.6mm")
@@
 	(footprint "Resistor_THT:R_Axial_DIN0204_L3.6mm_D1.6mm_P5.08mm_Horizontal"
 		(layer "F.Cu")
-		(at 129 120.54 90)
+		(at 128 114.08 90)
 		(descr "Resistor, Axial_DIN0204 series, Axial, Horizontal, pin pitch=5.08mm, 0.167W, length*diameter=3.6*1.6mm^2, http://cdn-reichelt.de/documents/datenblatt/B400/1_4W%23YAG.pdf")
 		(tags "Resistor Axial_DIN0204 series Axial Horizontal pin pitch 5.08mm 0.167W length 3.6mm diameter 1.6mm")
@@
 	(footprint "Resistor_THT:R_Axial_DIN0204_L3.6mm_D1.6mm_P5.08mm_Horizontal"
 		(layer "F.Cu")
-		(at 157.555 111.975)
+		(at 139.92 108)
 		(descr "Resistor, Axial_DIN0204 series, Axial, Horizontal, pin pitch=5.08mm, 0.167W, length*diameter=3.6*1.6mm^2, http://cdn-reichelt.de/documents/datenblatt/B400/1_4W%23YAG.pdf")
 		(tags "Resistor Axial_DIN0204 series Axial Horizontal pin pitch 5.08mm 0.167W length 3.6mm diameter 1.6mm")
@@
 	(footprint "Resistor_THT:R_Axial_DIN0204_L3.6mm_D1.6mm_P5.08mm_Horizontal"
 		(layer "F.Cu")
-		(at 157.555 116.975)
+		(at 139 113)
 		(descr "Resistor, Axial_DIN0204 series, Axial, Horizontal, pin pitch=5.08mm, 0.167W, length*diameter=3.6*1.6mm^2, http://cdn-reichelt.de/documents/datenblatt/B400/1_4W%23YAG.pdf")
 		(tags "Resistor Axial_DIN0204 series Axial Horizontal pin pitch 5.08mm 0.167W length 3.6mm diameter 1.6mm")
@@
 	(footprint "Resistor_THT:R_Axial_DIN0204_L3.6mm_D1.6mm_P5.08mm_Horizontal"
 		(layer "F.Cu")
-		(at 141.08 117)
+		(at 130.92 119)
 		(descr "Resistor, Axial_DIN0204 series, Axial, Horizontal, pin pitch=5.08mm, 0.167W, length*diameter=3.6*1.6mm^2, http://cdn-reichelt.de/documents/datenblatt/B400/1_4W%23YAG.pdf")
 		(tags "Resistor Axial_DIN0204 series Axial Horizontal pin pitch 5.08mm 0.167W length 3.6mm diameter 1.6mm")
@@
 	(footprint "Resistor_THT:R_Axial_DIN0204_L3.6mm_D1.6mm_P5.08mm_Horizontal"
 		(layer "F.Cu")
-		(at 158.015 120.975)
+		(at 139 116)
 		(descr "Resistor, Axial_DIN0204 series, Axial, Horizontal, pin pitch=5.08mm, 0.167W, length*diameter=3.6*1.6mm^2, http://cdn-reichelt.de/documents/datenblatt/B400/1_4W%23YAG.pdf")
 		(tags "Resistor Axial_DIN0204 series Axial Horizontal pin pitch 5.08mm 0.167W length 3.6mm diameter 1.6mm")
@@
 	(footprint "Resistor_THT:R_Axial_DIN0204_L3.6mm_D1.6mm_P5.08mm_Horizontal"
 		(layer "F.Cu")
-		(at 146 108)
+		(at 151 113)
 		(descr "Resistor, Axial_DIN0204 series, Axial, Horizontal, pin pitch=5.08mm, 0.167W, length*diameter=3.6*1.6mm^2, http://cdn-reichelt.de/documents/datenblatt/B400/1_4W%23YAG.pdf")
 		(tags "Resistor Axial_DIN0204 series Axial Horizontal pin pitch 5.08mm 0.167W length 3.6mm diameter 1.6mm")
@@
 	(footprint "Package_SO:SOIC-14_3.9x8.7mm_P1.27mm"
 		(layer "F.Cu")
-		(at 138.46 109.475 -90)
+		(at 135 106 -90)
 		(descr "SOIC, 14 Pin (JEDEC MS-012AB, https://www.analog.com/media/en/package-pcb-resources/package/pkg_pdf/soic_narrow-r/r_14.pdf), generated with kicad-footprint-generator ipc_gullwing_generator.py")
 		(tags "SOIC SO")
@@
 		)
 		(fp_text user "${REFERENCE}"
-			(at 0 0 0)
+			(at 0.525 0.46 0)
 			(layer "F.Fab")
 			(effects
@@
 	(footprint "Resistor_THT:R_Axial_DIN0204_L3.6mm_D1.6mm_P5.08mm_Horizontal"
 		(layer "F.Cu")
-		(at 133 117)
+		(at 130.92 122)
 		(descr "Resistor, Axial_DIN0204 series, Axial, Horizontal, pin pitch=5.08mm, 0.167W, length*diameter=3.6*1.6mm^2, http://cdn-reichelt.de/documents/datenblatt/B400/1_4W%23YAG.pdf")
 		(tags "Resistor Axial_DIN0204 series Axial Horizontal pin pitch 5.08mm 0.167W length 3.6mm diameter 1.6mm")
@@
 	(footprint "Resistor_THT:R_Axial_DIN0204_L3.6mm_D1.6mm_P5.08mm_Horizontal"
 		(layer "F.Cu")
-		(at 149.46 117)
+		(at 130.92 113)
 		(descr "Resistor, Axial_DIN0204 series, Axial, Horizontal, pin pitch=5.08mm, 0.167W, length*diameter=3.6*1.6mm^2, http://cdn-reichelt.de/documents/datenblatt/B400/1_4W%23YAG.pdf")
 		(tags "Resistor Axial_DIN0204 series Axial Horizontal pin pitch 5.08mm 0.167W length 3.6mm diameter 1.6mm")
@@
 	(footprint "Resistor_THT:R_Axial_DIN0204_L3.6mm_D1.6mm_P5.08mm_Horizontal"
 		(layer "F.Cu")
-		(at 129 96 -90)
+		(at 128 95 -90)
 		(descr "Resistor, Axial_DIN0204 series, Axial, Horizontal, pin pitch=5.08mm, 0.167W, length*diameter=3.6*1.6mm^2, http://cdn-reichelt.de/documents/datenblatt/B400/1_4W%23YAG.pdf")
 		(tags "Resistor Axial_DIN0204 series Axial Horizontal pin pitch 5.08mm 0.167W length 3.6mm diameter 1.6mm")
@@
 		)
 		(fp_text user "${REFERENCE}"
-			(at 2.54 0 90)
+			(at 1 1 90)
 			(layer "F.Fab")
 			(effects
@@
 	(footprint "Resistor_THT:R_Axial_DIN0204_L3.6mm_D1.6mm_P5.08mm_Horizontal"
 		(layer "F.Cu")
-		(at 132.92 101)
+		(at 132 99)
 		(descr "Resistor, Axial_DIN0204 series, Axial, Horizontal, pin pitch=5.08mm, 0.167W, length*diameter=3.6*1.6mm^2, http://cdn-reichelt.de/documents/datenblatt/B400/1_4W%23YAG.pdf")
 		(tags "Resistor Axial_DIN0204 series Axial Horizontal pin pitch 5.08mm 0.167W length 3.6mm diameter 1.6mm")
@@
 	(footprint "Resistor_THT:R_Axial_DIN0204_L3.6mm_D1.6mm_P5.08mm_Horizontal"
 		(layer "F.Cu")
-		(at 129 111.08 90)
+		(at 128 107.08 90)
 		(descr "Resistor, Axial_DIN0204 series, Axial, Horizontal, pin pitch=5.08mm, 0.167W, length*diameter=3.6*1.6mm^2, http://cdn-reichelt.de/documents/datenblatt/B400/1_4W%23YAG.pdf")
 		(tags "Resistor Axial_DIN0204 series Axial Horizontal pin pitch 5.08mm 0.167W length 3.6mm diameter 1.6mm")
@@
 	(footprint "Connector_PinSocket_2.54mm:PinSocket_1x02_P2.54mm_Vertical"
 		(layer "F.Cu")
-		(at 140.46 96 90)
+		(at 131 95 90)
 		(descr "Through hole straight socket strip, 1x02, 2.54mm pitch, single row (from Kicad 4.0.7), script generated")
 		(tags "Through hole socket strip THT 1x02 2.54mm single row")
@@
 	(gr_rect
 		(start 114 93)
-		(end 204 126)
+		(end 202 126)
 		(stroke
 			(width 0.05)
-			(type default)
+			(type solid)
 		)
 		(fill no)

Commit message: pcb update
Parts:
- moved R13 30.1 mm to (159.9, 105.0)
- moved R20 26.4 mm to (161.9, 121.0)
- moved R21 25.6 mm to (160.5, 113.0)
- moved R19 24.6 mm to (161.9, 96.0)
- moved D3 24.4 mm to (172.0, 125.0)
- moved R22 24.2 mm to (129.9, 116.0)
- moved D2 22.0 mm to (172.0, 112.0)
- moved R12 22.0 mm to (149.9, 105.0)
- moved D1 21.9 mm to (172.0, 98.5)
- moved J8 18.5 mm to (151.0, 119.0)
- moved R15 18.3 mm to (139.9, 99.0)
- moved R14 18.1 mm to (139.9, 102.0)
- moved J9 17.8 mm to (151.0, 124.0)
- moved J7 17.3 mm to (151.0, 114.0)
- moved J5 17.1 mm to (151.1, 96.0)
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Other:
- board size 88 x 33 mm -> 66 x 37 mm

Commit message: light_maze_pcb_edit
Parts:
- moved D1 47.7 mm to (131.0, 123.0), turned to 0 degrees
- moved R19 39.3 mm to (130.0, 119.0)
- moved D2 36.7 mm to (137.0, 123.0), turned to 0 degrees
- moved D3 29.1 mm to (143.0, 123.0), turned to 0 degrees
- moved R21 16.1 mm to (151.0, 126.0)
- moved R20 13.6 mm to (150.9, 129.0)
- moved R13 12.4 mm to (147.5, 106.0)
- moved J4 4.00 mm to (156.9, 109.0), turned to 180 degrees
- moved R12 3.11 mm to (147.5, 103.0)
- moved J3 3.00 mm to (148.0, 109.0)
- moved J2 2.08 mm to (138.9, 109.0)
- moved J6 2.00 mm to (150.9, 99.0)
- moved J9 2.00 mm to (150.9, 122.0)
- moved J1 2.00 mm to (141.5, 95.0)
- moved J5 1.00 mm to (151.0, 95.0)
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Other:
- board size 66 x 37 mm -> 45 x 39 mm

Commit message: PCB routing
Routing:
- net ground: track 0.00 -> 130.3 mm
- net Vcc: track 0.00 -> 108.8 mm
- net x: track 0.00 -> 49.1 mm, vias 0 -> 1
- net Net-(U2C-+): track 0.00 -> 34.6 mm, vias 0 -> 1
- net c: track 0.00 -> 33.1 mm
- net f: track 0.00 -> 25.0 mm
- net Net-(U2B-+): track 0.00 -> 24.3 mm
- net b: track 0.00 -> 22.5 mm
- net a: track 0.00 -> 22.2 mm
- net Net-(U2A-+): track 0.00 -> 20.0 mm
- net Net-(D2-A): track 0.00 -> 19.3 mm
- net y: track 0.00 -> 17.1 mm
- net Net-(U2A--): track 0.00 -> 16.0 mm
- net Net-(J5-Pin_2): track 0.00 -> 15.3 mm
- net Net-(J9-Pin_2): track 0.00 -> 14.8 mm
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